Commit message: Twin: real UFACTORY 850 geometry from the official STEP
- simulation/assets/uf850/link_base..link6.stl: the seven FX85 parts of
  'UFACTORY 850(FX8510)-20260626.STEP', each moved into its URDF link frame
  (checked against UFACTORY's xarm_description meshes: joints at 0 deg within
  0.06 deg, surfaces within a median of 0.6 mm).
- step_to_link_meshes.py regenerates them from a STEP.
- primitive_arm.py draws the arms with these meshes when present; collision
  shapes stay primitive.

Co-Authored-By: Claude Opus 5.5 <noreply@anthropic.com>
Claude-Session: https://claude.ai/code/session_01BipZG4PRuhm1rMCJYajyai

File: simulation/assets_generated/primitive_xarm850_left.urdf (robot description, URDF)
Before this commit: robot uf850_primitive, 9 links, 8 joints
Links:
- link link1: geometry visual mesh filename=../assets/uf850/link1.stl scale=1 1 1
- link link2: geometry collision cylinder length=0.3900 radius=0.0450; visual mesh filename=../assets/uf850/link2.stl scale=1 1 1
- link link3: geometry collision cylinder length=0.4516 radius=0.0450; visual mesh filename=../assets/uf850/link3.stl scale=1 1 1
- link link4: geometry visual mesh filename=../assets/uf850/link4.stl scale=1 1 1
- link link5: geometry collision cylinder length=0.0900 radius=0.0450; visual mesh filename=../assets/uf850/link5.stl scale=1 1 1
- link link6: geometry visual mesh filename=../assets/uf850/link6.stl scale=1 1 1
- link link_base: geometry collision cylinder length=0.3640 radius=0.0550; visual mesh filename=../assets/uf850/link_base.stl scale=1 1 1
